Commit message: feat: update 3d printer with STL slicing, workspace validation, and test scripts
Add triangle prism STL/gcode resources, improve kinematics solver,
update URDF workcell models, and clean up build/install/log artifacts.

Co-Authored-By: Claude Opus 4.6 <noreply@anthropic.com>

File: workspace/src/ur_3d_printer/urdf/optical_table.urdf.xacro (robot description, xacro)
@@ -3,8 +3,15 @@
   <!-- Standalone mode argument -->
   <xacro:arg name="standalone" default="false"/>
+  <!-- surface_z: absolute z of the table top surface.  When the UR driver
+       publishes base_link at z=0, set surface_z=-0.02 so the robot's 2 cm
+       mounting plate sits flush on the table. -->
+  <xacro:arg name="surface_z" default="-0.02"/>
+  <!-- leg_height: visual length of the table legs (extends downward). -->
+  <xacro:arg name="leg_height" default="0.88"/>
   <!-- Table parameters -->
   <xacro:property name="table_length" value="1.2"/>
   <xacro:property name="table_width" value="0.8"/>
-  <xacro:property name="table_height" value="0.9"/>
+  <xacro:property name="surface_z" value="$(arg surface_z)"/>
+  <xacro:property name="leg_height" value="$(arg leg_height)"/>
   <xacro:property name="table_thickness" value="0.05"/>
   <xacro:property name="leg_size" value="0.06"/>
@@ -13,5 +20,5 @@
   <xacro:property name="grid_strip_width" value="0.003"/>
   <xacro:property name="grid_strip_height" value="0.002"/>
-  <xacro:property name="table_x_offset" value="0.15"/>
+  <xacro:property name="table_x_offset" value="-0.15"/>
   <!-- Materials -->
   <material name="brushed_aluminum">
@@ -39,5 +46,5 @@
       <parent link="${prefix}table_base_link"/>
       <child link="${prefix}table_top"/>
-      <origin xyz="0 0 ${table_height - table_thickness/2}" rpy="0 0 0"/>
+      <origin xyz="0 0 ${surface_z - table_thickness/2}" rpy="0 0 0"/>
     </joint>
     <link name="${prefix}table_top">
@@ -137,10 +144,10 @@
         <parent link="${prefix}table_base_link"/>
         <child link="${prefix}${name}"/>
-        <origin xyz="${x} ${y} ${(table_height - table_thickness)/2}" rpy="0 0 0"/>
+        <origin xyz="${x} ${y} ${surface_z - table_thickness - leg_height/2}" rpy="0 0 0"/>
       </joint>
       <link name="${prefix}${name}">
         <visual>
           <geometry>
-            <box size="${leg_size} ${leg_size} ${table_height - table_thickness}"/>
+            <box size="${leg_size} ${leg_size} ${leg_height}"/>
           </geometry>
           <material name="dark_steel"/>
@@ -148,5 +155,5 @@
         <collision>
           <geometry>
-            <box size="${leg_size} ${leg_size} ${table_height - table_thickness}"/>
+            <box size="${leg_size} ${leg_size} ${leg_height}"/>
           </geometry>
         </collision>

File: workspace/src/ur_3d_printer/urdf/print_bed.urdf.xacro (robot description, xacro)
@@ -2,4 +2,5 @@
 <robot xmlns:xacro="http://www.ros.org/wiki/xacro" name="print_bed">
   <xacro:arg name="standalone" default="false"/>
+  <xacro:arg name="bed_z" default="-0.01"/>
   <!-- Print Bed Parameters -->
   <xacro:arg name="bed_width" default="0.3"/>      <!-- X dimension (m) -->
@@ -16,5 +17,5 @@
     <color rgba="0.4 0.4 0.4 1.0"/>
   </material>
-  <xacro:macro name="print_bed" params="parent prefix:='' x:=0.4 y:=0.0 z:=0.92">
+  <xacro:macro name="print_bed" params="parent prefix:='' x:=-0.3 y:=0.0 z:=0.005">
     <!-- Bed mount to world/table -->
     <joint name="${prefix}print_bed_joint" type="fixed">
@@ -63,5 +64,5 @@
   <xacro:if value="$(arg standalone)">
     <link name="world"/>
-    <xacro:print_bed parent="world" prefix=""/>
+    <xacro:print_bed parent="world" prefix="" z="$(arg bed_z)"/>
   </xacro:if>
 </robot>
