Commit message: feat: add multi-model UR robot support and fix digital twin rendering
- Add all 6 UR models: UR3e, UR5e, UR10e, UR16e, UR20, UR30
- Generate per-model URDF with cross-model mesh path resolution
  (UR16e shares ur10e meshes, UR30 shares ur20 meshes)
- Copy DAE visual + STL collision meshes for all models
- Add robot model selector in Live panel and settings dropdown
- Fix URDF Z-up to Three.js Y-up rotation (-90° X)
- Align grid and table surface at robot mount height (0.9m)
- Clean URDFs: strip ros2_control/gazebo/transmission tags
- Robot model selection persists via localStorage

Co-Authored-By: Claude Opus 4.6 (1M context) <noreply@anthropic.com>

File: workspace/src/ur_3d_printer_web/frontend/public/robots/ur10e.urdf (robot description, URDF)
Before this commit: robot ur_3d_printer_cell, 20 links, 19 joints
Links:
- link base_link_inertia: geometry collision mesh filename=/meshes/ur10e/base.stl; visual mesh filename=/meshes/ur10e/base.dae
- link forearm_link: mass 2.846 -> 3.989; geometry collision mesh filename=/meshes/ur10e/forearm.stl; visual mesh filename=/meshes/ur10e/forearm.dae
- link shoulder_link: mass 3.761 -> 7.369; geometry collision mesh filename=/meshes/ur10e/shoulder.stl; visual mesh filename=/meshes/ur10e/shoulder.dae
- link upper_arm_link: mass 8.058 -> 13.051; geometry collision mesh filename=/meshes/ur10e/upperarm.stl; visual mesh filename=/meshes/ur10e/upperarm.dae
- link wrist_1_link: mass 1.37 -> 2.1; geometry collision mesh filename=/meshes/ur10e/wrist1.stl; visual mesh filename=/meshes/ur10e/wrist1.dae
- link wrist_2_link: mass 1.3 -> 1.98; geometry collision mesh filename=/meshes/ur10e/wrist2.stl; visual mesh filename=/meshes/ur10e/wrist2.dae
- link wrist_3_link: mass 0.365 -> 0.615; geometry collision mesh filename=/meshes/ur10e/wrist3.stl; visual mesh filename=/meshes/ur10e/wrist3.dae
Joints:
- joint elbow_joint: origin xyz=-0.425 0 0 rpy=0 0 0 -> xyz=-0.6127 0 0 rpy=0 0 0
- joint shoulder_lift_joint: limit lower=-6.283185307179586 upper=6.283185307179586 effort=150.0 velocity=3.141592653589793 -> lower=-6.283185307179586 upper=6.283185307179586 effort=330.0 velocity=2.0943951023931953
- joint shoulder_pan_joint: limit lower=-6.283185307179586 upper=6.283185307179586 effort=150.0 velocity=3.141592653589793 -> lower=-6.283185307179586 upper=6.283185307179586 effort=330.0 velocity=2.0943951023931953; origin xyz=0 0 0.1625 rpy=0 0 0 -> xyz=0 0 0.1807 rpy=0 0 0
- joint wrist_1_joint: limit lower=-6.283185307179586 upper=6.283185307179586 effort=28.0 velocity=3.141592653589793 -> lower=-6.283185307179586 upper=6.283185307179586 effort=54.0 velocity=3.141592653589793; origin xyz=-0.3922 0 0.1333 rpy=0 0 0 -> xyz=-0.57155 0 0.17415 rpy=0 0 0
- joint wrist_2_joint: limit lower=-6.283185307179586 upper=6.283185307179586 effort=28.0 velocity=3.141592653589793 -> lower=-6.283185307179586 upper=6.283185307179586 effort=54.0 velocity=3.141592653589793; origin xyz=0 -0.0997 -2.044881182297852e-11 rpy=1.570796327 0 0 -> xyz=0 -0.11985 -2.458164590756244e-11 rpy=1.570796327 0 0
- joint wrist_3_joint: limit lower=-6.283185307179586 upper=6.283185307179586 effort=28.0 velocity=3.141592653589793 -> lower=-6.283185307179586 upper=6.283185307179586 effort=54.0 velocity=3.141592653589793; origin xyz=0 0.0996 -2.042830148012698e-11 rpy=1.570796326589793 3.141592653589793 3.141592653589793 -> xyz=0 0.11655 -2.390480459346185e-11 rpy=1.570796326589793 3.141592653589793 3.141592653589793

File: workspace/src/ur_3d_printer_web/frontend/public/robots/ur16e.urdf (robot description, URDF)
Before this commit: robot ur_3d_printer_cell, 20 links, 19 joints
Links:
- link base_link_inertia: geometry collision mesh filename=/meshes/ur10e/base.stl; visual mesh filename=/meshes/ur10e/base.dae
- link forearm_link: mass 2.846 -> 4.321; geometry collision mesh filename=/meshes/ur16e/forearm.stl; visual mesh filename=/meshes/ur16e/forearm.dae
- link shoulder_link: mass 3.761 -> 7.369; geometry collision mesh filename=/meshes/ur10e/shoulder.stl; visual mesh filename=/meshes/ur10e/shoulder.dae
- link upper_arm_link: mass 8.058 -> 10.45; geometry collision mesh filename=/meshes/ur16e/upperarm.stl; visual mesh filename=/meshes/ur16e/upperarm.dae
- link wrist_1_link: mass 1.37 -> 2.18; geometry collision mesh filename=/meshes/ur10e/wrist1.stl; visual mesh filename=/meshes/ur10e/wrist1.dae
- link wrist_2_link: mass 1.3 -> 2.033; geometry collision mesh filename=/meshes/ur10e/wrist2.stl; visual mesh filename=/meshes/ur10e/wrist2.dae
- link wrist_3_link: mass 0.365 -> 0.907; geometry collision mesh filename=/meshes/ur10e/wrist3.stl; visual mesh filename=/meshes/ur10e/wrist3.dae
Joints:
- joint elbow_joint: origin xyz=-0.425 0 0 rpy=0 0 0 -> xyz=-0.4784 0 0 rpy=0 0 0
- joint shoulder_lift_joint: limit lower=-6.283185307179586 upper=6.283185307179586 effort=150.0 velocity=3.141592653589793 -> lower=-6.283185307179586 upper=6.283185307179586 effort=330.0 velocity=2.0943951023931953
- joint shoulder_pan_joint: limit lower=-6.283185307179586 upper=6.283185307179586 effort=150.0 velocity=3.141592653589793 -> lower=-6.283185307179586 upper=6.283185307179586 effort=330.0 velocity=2.0943951023931953; origin xyz=0 0 0.1625 rpy=0 0 0 -> xyz=0 0 0.1807 rpy=0 0 0
- joint wrist_1_joint: limit lower=-6.283185307179586 upper=6.283185307179586 effort=28.0 velocity=3.141592653589793 -> lower=-6.283185307179586 upper=6.283185307179586 effort=54.0 velocity=3.141592653589793; origin xyz=-0.3922 0 0.1333 rpy=0 0 0 -> xyz=-0.36 0 0.17415 rpy=0 0 0
- joint wrist_2_joint: limit lower=-6.283185307179586 upper=6.283185307179586 effort=28.0 velocity=3.141592653589793 -> lower=-6.283185307179586 upper=6.283185307179586 effort=54.0 velocity=3.141592653589793; origin xyz=0 -0.0997 -2.044881182297852e-11 rpy=1.570796327 0 0 -> xyz=0 -0.11985 -2.458164590756244e-11 rpy=1.570796327 0 0
- joint wrist_3_joint: limit lower=-6.283185307179586 upper=6.283185307179586 effort=28.0 velocity=3.141592653589793 -> lower=-6.283185307179586 upper=6.283185307179586 effort=54.0 velocity=3.141592653589793; origin xyz=0 0.0996 -2.042830148012698e-11 rpy=1.570796326589793 3.141592653589793 3.141592653589793 -> xyz=0 0.11655 -2.390480459346185e-11 rpy=1.570796326589793 3.141592653589793 3.141592653589793

File: workspace/src/ur_3d_printer_web/frontend/public/robots/ur20.urdf (robot description, URDF)
Before this commit: robot ur_3d_printer_cell, 20 links, 19 joints
Links:
- link base_link_inertia: geometry collision mesh filename=/meshes/ur20/base.stl; visual mesh filename=/meshes/ur20/base.dae
- link forearm_link: mass 2.846 -> 7.879; geometry collision mesh filename=/meshes/ur20/forearm.stl; visual mesh filename=/meshes/ur20/forearm.dae
- link shoulder_link: mass 3.761 -> 16.343; geometry collision mesh filename=/meshes/ur20/shoulder.stl; visual mesh filename=/meshes/ur20/shoulder.dae
- link upper_arm_link: mass 8.058 -> 29.632; geometry collision mesh filename=/meshes/ur20/upperarm.stl; visual mesh filename=/meshes/ur20/upperarm.dae
- link wrist_1_link: mass 1.37 -> 3.054; geometry collision mesh filename=/meshes/ur20/wrist1.stl; visual mesh filename=/meshes/ur20/wrist1.dae
- link wrist_2_link: mass 1.3 -> 3.126; geometry collision mesh filename=/meshes/ur20/wrist2.stl; visual mesh filename=/meshes/ur20/wrist2.dae
- link wrist_3_link: mass 0.365 -> 0.926; geometry collision mesh filename=/meshes/ur20/wrist3.stl; visual mesh filename=/meshes/ur20/wrist3.dae
Joints:
- joint elbow_joint: limit lower=-3.141592653589793 upper=3.141592653589793 effort=150.0 velocity=3.141592653589793 -> lower=-3.141592653589793 upper=3.141592653589793 effort=433.0 velocity=2.6179938779914944; origin xyz=-0.425 0 0 rpy=0 0 0 -> xyz=-0.862 0 0 rpy=0 0 0
- joint shoulder_lift_joint: limit lower=-6.283185307179586 upper=6.283185307179586 effort=150.0 velocity=3.141592653589793 -> lower=-6.283185307179586 upper=6.283185307179586 effort=738.0 velocity=2.0943951023931953
- joint shoulder_pan_joint: limit lower=-6.283185307179586 upper=6.283185307179586 effort=150.0 velocity=3.141592653589793 -> lower=-6.283185307179586 upper=6.283185307179586 effort=738.0 velocity=2.0943951023931953; origin xyz=0 0 0.1625 rpy=0 0 0 -> xyz=0 0 0.2363 rpy=0 0 0
- joint wrist_1_joint: limit lower=-6.283185307179586 upper=6.283185307179586 effort=28.0 velocity=3.141592653589793 -> lower=-6.283185307179586 upper=6.283185307179586 effort=107.0 velocity=3.6651914291880923; origin xyz=-0.3922 0 0.1333 rpy=0 0 0 -> xyz=-0.7287 0 0.201 rpy=0 0 0
- joint wrist_2_joint: limit lower=-6.283185307179586 upper=6.283185307179586 effort=28.0 velocity=3.141592653589793 -> lower=-6.283185307179586 upper=6.283185307179586 effort=107.0 velocity=3.6651914291880923; origin xyz=0 -0.0997 -2.044881182297852e-11 rpy=1.570796327 0 0 -> xyz=0 -0.1593 -3.267297616249225e-11 rpy=1.570796327 0 0
- joint wrist_3_joint: limit lower=-6.283185307179586 upper=6.283185307179586 effort=28.0 velocity=3.141592653589793 -> lower=-6.283185307179586 upper=6.283185307179586 effort=107.0 velocity=3.6651914291880923; origin xyz=0 0.0996 -2.042830148012698e-11 rpy=1.570796326589793 3.141592653589793 3.141592653589793 -> xyz=0 0.1543 -3.1647459019915597e-11 rpy=1.570796326589793 3.141592653589793 3.141592653589793

File: workspace/src/ur_3d_printer_web/frontend/public/robots/ur30.urdf (robot description, URDF)
Before this commit: robot ur_3d_printer_cell, 20 links, 19 joints
Links:
- link base_link_inertia: geometry collision mesh filename=/meshes/ur20/base.stl; visual mesh filename=/meshes/ur20/base.dae
- link forearm_link: mass 2.846 -> 7.156; geometry collision mesh filename=/meshes/ur30/forearm.stl; visual mesh filename=/meshes/ur30/forearm.dae
- link shoulder_link: mass 3.761 -> 16.343; geometry collision mesh filename=/meshes/ur20/shoulder.stl; visual mesh filename=/meshes/ur20/shoulder.dae
- link upper_arm_link: mass 8.058 -> 28.542; geometry collision mesh filename=/meshes/ur30/upperarm.stl; visual mesh filename=/meshes/ur30/upperarm.dae
- link wrist_1_link: mass 1.37 -> 3.054; geometry collision mesh filename=/meshes/ur20/wrist1.stl; visual mesh filename=/meshes/ur20/wrist1.dae
- link wrist_2_link: mass 1.3 -> 3.126; geometry collision mesh filename=/meshes/ur20/wrist2.stl; visual mesh filename=/meshes/ur20/wrist2.dae
- link wrist_3_link: mass 0.365 -> 0.926; geometry collision mesh filename=/meshes/ur20/wrist3.stl; visual mesh filename=/meshes/ur20/wrist3.dae
Joints:
- joint elbow_joint: limit lower=-3.141592653589793 upper=3.141592653589793 effort=150.0 velocity=3.141592653589793 -> lower=-3.141592653589793 upper=3.141592653589793 effort=433.0 velocity=2.6179938779914944; origin xyz=-0.425 0 0 rpy=0 0 0 -> xyz=-0.637 0 0 rpy=0 0 0
- joint shoulder_lift_joint: limit lower=-6.283185307179586 upper=6.283185307179586 effort=150.0 velocity=3.141592653589793 -> lower=-6.283185307179586 upper=6.283185307179586 effort=738.0 velocity=2.0943951023931953
- joint shoulder_pan_joint: limit lower=-6.283185307179586 upper=6.283185307179586 effort=150.0 velocity=3.141592653589793 -> lower=-6.283185307179586 upper=6.283185307179586 effort=738.0 velocity=2.0943951023931953; origin xyz=0 0 0.1625 rpy=0 0 0 -> xyz=0 0 0.2363 rpy=0 0 0
- joint wrist_1_joint: limit lower=-6.283185307179586 upper=6.283185307179586 effort=28.0 velocity=3.141592653589793 -> lower=-6.283185307179586 upper=6.283185307179586 effort=107.0 velocity=3.6651914291880923; origin xyz=-0.3922 0 0.1333 rpy=0 0 0 -> xyz=-0.5037 0 0.201 rpy=0 0 0
- joint wrist_2_joint: limit lower=-6.283185307179586 upper=6.283185307179586 effort=28.0 velocity=3.141592653589793 -> lower=-6.283185307179586 upper=6.283185307179586 effort=107.0 velocity=3.6651914291880923; origin xyz=0 -0.0997 -2.044881182297852e-11 rpy=1.570796327 0 0 -> xyz=0 -0.1593 -3.267297616249225e-11 rpy=1.570796327 0 0
- joint wrist_3_joint: limit lower=-6.283185307179586 upper=6.283185307179586 effort=28.0 velocity=3.141592653589793 -> lower=-6.283185307179586 upper=6.283185307179586 effort=107.0 velocity=3.6651914291880923; origin xyz=0 0.0996 -2.042830148012698e-11 rpy=1.570796326589793 3.141592653589793 3.141592653589793 -> xyz=0 0.1543 -3.1647459019915597e-11 rpy=1.570796326589793 3.141592653589793 3.141592653589793

File: workspace/src/ur_3d_printer_web/frontend/public/robots/ur3e.urdf (robot description, URDF)
Before this commit: robot ur_3d_printer_cell, 20 links, 19 joints
Links:
- link base_link_inertia: mass 4.0 -> 2.0; geometry collision mesh filename=/meshes/ur3e/base.stl; visual mesh filename=/meshes/ur3e/base.dae
- link forearm_link: mass 2.846 -> 1.437; geometry collision mesh filename=/meshes/ur3e/forearm.stl; visual mesh filename=/meshes/ur3e/forearm.dae
- link shoulder_link: mass 3.761 -> 1.98; geometry collision mesh filename=/meshes/ur3e/shoulder.stl; visual mesh filename=/meshes/ur3e/shoulder.dae
- link upper_arm_link: mass 8.058 -> 3.4445; geometry collision mesh filename=/meshes/ur3e/upperarm.stl; visual mesh filename=/meshes/ur3e/upperarm.dae
- link wrist_1_link: mass 1.37 -> 0.871; geometry collision mesh filename=/meshes/ur3e/wrist1.stl; visual mesh filename=/meshes/ur3e/wrist1.dae
- link wrist_2_link: mass 1.3 -> 0.805; geometry collision mesh filename=/meshes/ur3e/wrist2.stl; visual mesh filename=/meshes/ur3e/wrist2.dae
- link wrist_3_link: mass 0.365 -> 0.261; geometry collision mesh filename=/meshes/ur3e/wrist3.stl; visual mesh filename=/meshes/ur3e/wrist3.dae
Joints:
- joint elbow_joint: limit lower=-3.141592653589793 upper=3.141592653589793 effort=150.0 velocity=3.141592653589793 -> lower=-3.141592653589793 upper=3.141592653589793 effort=28.0 velocity=3.141592653589793; origin xyz=-0.425 0 0 rpy=0 0 0 -> xyz=-0.24355 0 0 rpy=0 0 0
- joint shoulder_lift_joint: limit lower=-6.283185307179586 upper=6.283185307179586 effort=150.0 velocity=3.141592653589793 -> lower=-6.283185307179586 upper=6.283185307179586 effort=54.0 velocity=3.141592653589793
- joint shoulder_pan_joint: limit lower=-6.283185307179586 upper=6.283185307179586 effort=150.0 velocity=3.141592653589793 -> lower=-6.283185307179586 upper=6.283185307179586 effort=54.0 velocity=3.141592653589793; origin xyz=0 0 0.1625 rpy=0 0 0 -> xyz=0 0 0.15185 rpy=0 0 0
- joint wrist_1_joint: limit lower=-6.283185307179586 upper=6.283185307179586 effort=28.0 velocity=3.141592653589793 -> lower=-6.283185307179586 upper=6.283185307179586 effort=9.0 velocity=6.283185307179586; origin xyz=-0.3922 0 0.1333 rpy=0 0 0 -> xyz=-0.2132 0 0.13105 rpy=0 0 0
- joint wrist_2_joint: limit lower=-6.283185307179586 upper=6.283185307179586 effort=28.0 velocity=3.141592653589793 -> lower=-6.283185307179586 upper=6.283185307179586 effort=9.0 velocity=6.283185307179586; origin xyz=0 -0.0997 -2.044881182297852e-11 rpy=1.570796327 0 0 -> xyz=0 -0.08535 -1.750557762378351e-11 rpy=1.570796327 0 0
- joint wrist_3_joint: limit lower=-6.283185307179586 upper=6.283185307179586 effort=28.0 velocity=3.141592653589793 -> effort=9.0 velocity=6.283185307179586; origin xyz=0 0.0996 -2.042830148012698e-11 rpy=1.570796326589793 3.141592653589793 3.141592653589793 -> xyz=0 0.0921 -1.8890025766262e-11 rpy=1.570796326589793 3.141592653589793 3.141592653589793; type revolute -> continuous

Commit message: fix: toolpath rendering, slicer layer transitions, digital twin pose, and bed position
- Toolpath: replace CatmullRomCurve3 with LineCurve3 segments to fix
  holes from spline overshoot, use FrontSide rendering, filter
  near-duplicate points
- Slicer: combine G0 X Y Z for layer transitions instead of separate
  G0 Z + G0 XY moves, so trajectory planner handles them as one segment
- Trajectory planner: add LOWER waypoint after HOVER in z-hop sequence
  for clean vertical descent between layers
- STL preview: solid meshPhysicalMaterial instead of transparent
  (eliminates see-through holes)
- Digital twin: normalize joint angles with atan2 + prefer +pi over -pi,
  ignoreLimits on URDF joints, fix bed position to x=-0.3 matching
  print_origin, add table with legs in Live view
- Docker compose: fix driver startup sequence — start ROS2 driver first,
  wait for port 50002, then play ExternalControl
- Bridge: add HTTP bridge endpoints for joint states, print state, and
  progress for host-mode development

Co-Authored-By: Claude Opus 4.6 (1M context) <noreply@anthropic.com>

File: workspace/src/ur_3d_printer_web/frontend/public/robots/ur10e.urdf (robot description, URDF)
Before this commit: robot ur_3d_printer_cell, 20 links, 19 joints
Joints:
- joint print_bed_joint: origin xyz=0.4 0.0 0.925 rpy=0 0 0 -> xyz=-0.3 0.0 0.925 rpy=0 0 0

File: workspace/src/ur_3d_printer_web/frontend/public/robots/ur16e.urdf (robot description, URDF)
Before this commit: robot ur_3d_printer_cell, 20 links, 19 joints
Joints:
- joint print_bed_joint: origin xyz=0.4 0.0 0.925 rpy=0 0 0 -> xyz=-0.3 0.0 0.925 rpy=0 0 0

File: workspace/src/ur_3d_printer_web/frontend/public/robots/ur20.urdf (robot description, URDF)
Before this commit: robot ur_3d_printer_cell, 20 links, 19 joints
Joints:
- joint print_bed_joint: origin xyz=0.4 0.0 0.925 rpy=0 0 0 -> xyz=-0.3 0.0 0.925 rpy=0 0 0

File: workspace/src/ur_3d_printer_web/frontend/public/robots/ur30.urdf (robot description, URDF)
Before this commit: robot ur_3d_printer_cell, 20 links, 19 joints
Joints:
- joint print_bed_joint: origin xyz=0.4 0.0 0.925 rpy=0 0 0 -> xyz=-0.3 0.0 0.925 rpy=0 0 0

File: workspace/src/ur_3d_printer_web/frontend/public/robots/ur3e.urdf (robot description, URDF)
Before this commit: robot ur_3d_printer_cell, 20 links, 19 joints
Joints:
- joint print_bed_joint: origin xyz=0.4 0.0 0.925 rpy=0 0 0 -> xyz=-0.3 0.0 0.925 rpy=0 0 0

File: workspace/src/ur_3d_printer_web/frontend/public/robots/ur5e.urdf (robot description, URDF)
Before this commit: robot ur_3d_printer_cell, 20 links, 19 joints
Joints:
- joint print_bed_joint: origin xyz=0.4 0.0 0.925 rpy=0 0 0 -> xyz=-0.3 0.0 0.925 rpy=0 0 0
