Commit message: feat: Mahor V5 PRO extruder 3D model in the web viewer and the cell URDF
Vendor STEP ("V5 PRO CAD") converted with FreeCAD and oriented for the
tool frame (motor back face on the flange at z=0, nozzle tip on +Z at
0.179 m, metres, 36k triangles):

- web: public/meshes/extruders/mahor_v5_pro.stl. The served URDFs now
  carry one mesh-based extruder_body link with placeholders that
  RobotModel fills from the backend's extruder_info (EXTRUDER_MESHES
  registry: model → mesh + tool length), replacing the box/cylinder FDM
  hotend. extruder_info is routed through the WebSocket into
  usePrintStore; ExtruderState types and the status card know the new
  HEATING / PURGING / FAULT states (i18n es/en).
- ROS: urdf/meshes/mahor_v5_pro.stl + urdf/pellet_extruder.urdf.xacro,
  selectable with extruder_type:=pellet (EXTRUDER_TYPE=pellet); nozzle_tcp
  at tool_length, which must match tool_offset_xyz in print_params.yaml.
- docs/EXTRUDERS.md: model provenance and regeneration steps.

Co-Authored-By: Claude Fable 5.1 <noreply@anthropic.com>

File: workspace/ur_3d_printer/urdf/ur_3d_printer_cell.urdf.xacro (robot description, xacro)
@@ -11,5 +11,5 @@
   <xacro:arg name="ur_type" default="ur5e"/>
   <xacro:arg name="tf_prefix" default=""/>
-  <xacro:arg name="extruder_type" default="fdm"/>  <!-- fdm or paste -->
+  <xacro:arg name="extruder_type" default="fdm"/>  <!-- fdm | paste | pellet (Mahor V5) -->
   <xacro:arg name="joint_limit_params" default="$(find ur_description)/config/$(arg ur_type)/joint_limits.yaml"/>
   <xacro:arg name="kinematics_params" default="$(find ur_description)/config/$(arg ur_type)/default_kinematics.yaml"/>
@@ -53,4 +53,5 @@
   <xacro:include filename="$(find ur_3d_printer)/urdf/fdm_extruder.urdf.xacro"/>
   <xacro:include filename="$(find ur_3d_printer)/urdf/paste_extruder.urdf.xacro"/>
+  <xacro:include filename="$(find ur_3d_printer)/urdf/pellet_extruder.urdf.xacro"/>
   <xacro:include filename="$(find ur_3d_printer)/urdf/print_bed.urdf.xacro"/>
   <xacro:property name="table_height" value="$(arg table_height)"/>
@@ -112,4 +113,7 @@
     <xacro:paste_extruder parent="$(arg tf_prefix)tool0" prefix="$(arg tf_prefix)"/>
   </xacro:if>
+  <xacro:if value="${'$(arg extruder_type)' == 'pellet'}">
+    <xacro:pellet_extruder parent="$(arg tf_prefix)tool0" prefix="$(arg tf_prefix)"/>
+  </xacro:if>
   <!-- Print Bed (conditional) -->
   <xacro:if value="$(arg include_bed)">

File: workspace/ur_3d_printer_web/frontend/public/robots/ur10e.urdf (robot description, URDF)
Before this commit: robot ur_3d_printer_cell, 20 links, 19 joints
Links:
- removed link extruder_heatbreak
- removed link extruder_heatsink
- removed link extruder_nozzle
- added link extruder_body; visual mesh filename=/meshes/extruders/__EXTRUDER_MESH__.stl
Joints:
- removed joint heatbreak_joint
- removed joint nozzle_joint
- joint extruder_base_joint: child extruder_heatsink -> extruder_body
- joint nozzle_tcp_joint: origin xyz=0 0 0.03 rpy=0 0 0 -> xyz=0 0 __TOOL_LENGTH__ rpy=0 0 0; parent extruder_nozzle -> extruder_body

File: workspace/ur_3d_printer_web/frontend/public/robots/ur16e.urdf (robot description, URDF)
Before this commit: robot ur_3d_printer_cell, 20 links, 19 joints
Links:
- removed link extruder_heatbreak
- removed link extruder_heatsink
- removed link extruder_nozzle
- added link extruder_body; visual mesh filename=/meshes/extruders/__EXTRUDER_MESH__.stl
Joints:
- removed joint heatbreak_joint
- removed joint nozzle_joint
- joint extruder_base_joint: child extruder_heatsink -> extruder_body
- joint nozzle_tcp_joint: origin xyz=0 0 0.03 rpy=0 0 0 -> xyz=0 0 __TOOL_LENGTH__ rpy=0 0 0; parent extruder_nozzle -> extruder_body

File: workspace/ur_3d_printer_web/frontend/public/robots/ur20.urdf (robot description, URDF)
Before this commit: robot ur_3d_printer_cell, 20 links, 19 joints
Links:
- removed link extruder_heatbreak
- removed link extruder_heatsink
- removed link extruder_nozzle
- added link extruder_body; visual mesh filename=/meshes/extruders/__EXTRUDER_MESH__.stl
Joints:
- removed joint heatbreak_joint
- removed joint nozzle_joint
- joint extruder_base_joint: child extruder_heatsink -> extruder_body
- joint nozzle_tcp_joint: origin xyz=0 0 0.03 rpy=0 0 0 -> xyz=0 0 __TOOL_LENGTH__ rpy=0 0 0; parent extruder_nozzle -> extruder_body

File: workspace/ur_3d_printer_web/frontend/public/robots/ur30.urdf (robot description, URDF)
Before this commit: robot ur_3d_printer_cell, 20 links, 19 joints
Links:
- removed link extruder_heatbreak
- removed link extruder_heatsink
- removed link extruder_nozzle
- added link extruder_body; visual mesh filename=/meshes/extruders/__EXTRUDER_MESH__.stl
Joints:
- removed joint heatbreak_joint
- removed joint nozzle_joint
- joint extruder_base_joint: child extruder_heatsink -> extruder_body
- joint nozzle_tcp_joint: origin xyz=0 0 0.03 rpy=0 0 0 -> xyz=0 0 __TOOL_LENGTH__ rpy=0 0 0; parent extruder_nozzle -> extruder_body

File: workspace/ur_3d_printer_web/frontend/public/robots/ur3e.urdf (robot description, URDF)
Before this commit: robot ur_3d_printer_cell, 20 links, 19 joints
Links:
- removed link extruder_heatbreak
- removed link extruder_heatsink
- removed link extruder_nozzle
- added link extruder_body; visual mesh filename=/meshes/extruders/__EXTRUDER_MESH__.stl
Joints:
- removed joint heatbreak_joint
- removed joint nozzle_joint
- joint extruder_base_joint: child extruder_heatsink -> extruder_body
- joint nozzle_tcp_joint: origin xyz=0 0 0.03 rpy=0 0 0 -> xyz=0 0 __TOOL_LENGTH__ rpy=0 0 0; parent extruder_nozzle -> extruder_body

File: workspace/ur_3d_printer_web/frontend/public/robots/ur5e.urdf (robot description, URDF)
Before this commit: robot ur_3d_printer_cell, 20 links, 19 joints
Links:
- removed link extruder_heatbreak
- removed link extruder_heatsink
- removed link extruder_nozzle
- added link extruder_body; visual mesh filename=/meshes/extruders/__EXTRUDER_MESH__.stl
Joints:
- removed joint heatbreak_joint
- removed joint nozzle_joint
- joint extruder_base_joint: child extruder_heatsink -> extruder_body
- joint nozzle_tcp_joint: origin xyz=0 0 0.03 rpy=0 0 0 -> xyz=0 0 __TOOL_LENGTH__ rpy=0 0 0; parent extruder_nozzle -> extruder_body
